File: PCB/tasarim_1_1.kicad_sch (KiCad schematic)
At the start: 51 parts, among them J1 SWD_Connector, J2 Boot_0, J3 LORA_Connector, J4 NRF_Connector, J5 ZW-21-08-L-T-200-157, J6 GPS_Connector, J7 Bootloader_Port, J8 APM_Connector, J9 Telemetri, SW1 SW_Push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

Commit message: new kicad version update
Parts:
- added unit 2 of J5
Connections:
- net GND: now also J5.03, J5.06, J5.09, J5.12, J5.15, J5.18, J5.21, J5.24, J5.27, J5.30, J5.33, J5.36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; no longer J5.03, J5.06, J5.09, J5.12, J5.15, J5.18, J5.21, J5.24, J5.27, J5.30, J5.33, J5.36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
